File: KF40-Micro-D_25_Double_Feedthrough/Double_MicroD_25_Gateway - Reversed/Double_MicroD_25_Gateway.kicad_pcb (KiCad board)
At the start: 4 copper layers, 37.4 x 37.4 mm, 4 parts, among them J1 DB25_Female, J2 DB25_Female, J3 DB25_Female, J4 DB25_Female

Commit message: updated kf40- reversed
Parts:
- turned J2 to 180 degrees
- turned J4 to 180 degrees
Connections:
- J2 pad 1: Net-(J1-Pad1) -> Net-(J1-Pad13)
- J2 pad 10: Net-(J1-Pad10) -> Net-(J1-Pad4)
- J2 pad 11: Net-(J1-Pad11) -> Net-(J1-Pad3)
- J2 pad 12: Net-(J1-Pad12) -> Net-(J1-Pad2)
- J2 pad 13: Net-(J1-Pad13) -> Net-(J1-Pad1)
- J2 pad 14: Net-(J1-Pad14) -> Net-(J1-Pad25)
- J2 pad 15: Net-(J1-Pad15) -> Net-(J1-Pad24)
- J2 pad 16: Net-(J1-Pad16) -> Net-(J1-Pad23)
- J2 pad 17: Net-(J1-Pad17) -> Net-(J1-Pad22)
- J2 pad 18: Net-(J1-Pad18) -> Net-(J1-Pad21)
- J2 pad 19: Net-(J1-Pad19) -> Net-(J1-Pad20)
- J2 pad 2: Net-(J1-Pad2) -> Net-(J1-Pad12)
- J2 pad 20: Net-(J1-Pad20) -> Net-(J1-Pad19)
- J2 pad 21: Net-(J1-Pad21) -> Net-(J1-Pad18)
- J2 pad 22: Net-(J1-Pad22) -> Net-(J1-Pad17)
- J2 pad 23: Net-(J1-Pad23) -> Net-(J1-Pad16)
- J2 pad 24: Net-(J1-Pad24) -> Net-(J1-Pad15)
- J2 pad 25: Net-(J1-Pad25) -> Net-(J1-Pad14)
- J2 pad 3: Net-(J1-Pad3) -> Net-(J1-Pad11)
- J2 pad 4: Net-(J1-Pad4) -> Net-(J1-Pad10)
- J2 pad 5: Net-(J1-Pad5) -> Net-(J1-Pad9)
- J2 pad 6: Net-(J1-Pad6) -> Net-(J1-Pad8)
- J2 pad 8: Net-(J1-Pad8) -> Net-(J1-Pad6)
- J2 pad 9: Net-(J1-Pad9) -> Net-(J1-Pad5)
- J4 pad 1: Net-(J3-Pad1) -> Net-(J3-Pad13)
- J4 pad 10: Net-(J3-Pad10) -> Net-(J3-Pad4)
- J4 pad 11: Net-(J3-Pad11) -> Net-(J3-Pad3)
- J4 pad 12: Net-(J3-Pad12) -> Net-(J3-Pad2)
- J4 pad 13: Net-(J3-Pad13) -> Net-(J3-Pad1)
- J4 pad 14: Net-(J3-Pad14) -> Net-(J3-Pad25)
- J4 pad 15: Net-(J3-Pad15) -> Net-(J3-Pad24)
- J4 pad 16: Net-(J3-Pad16) -> Net-(J3-Pad23)
- J4 pad 17: Net-(J3-Pad17) -> Net-(J3-Pad22)
- J4 pad 18: Net-(J3-Pad18) -> Net-(J3-Pad21)
- J4 pad 19: Net-(J3-Pad19) -> Net-(J3-Pad20)
- J4 pad 2: Net-(J3-Pad2) -> Net-(J3-Pad12)
- J4 pad 20: Net-(J3-Pad20) -> Net-(J3-Pad19)
- J4 pad 21: Net-(J3-Pad21) -> Net-(J3-Pad18)
- J4 pad 22: Net-(J3-Pad22) -> Net-(J3-Pad17)
- J4 pad 23: Net-(J3-Pad23) -> Net-(J3-Pad16)
- J4 pad 24: Net-(J3-Pad24) -> Net-(J3-Pad15)
- J4 pad 25: Net-(J3-Pad25) -> Net-(J3-Pad14)
- J4 pad 3: Net-(J3-Pad3) -> Net-(J3-Pad11)
- J4 pad 4: Net-(J3-Pad4) -> Net-(J3-Pad10)
- J4 pad 5: Net-(J3-Pad5) -> Net-(J3-Pad9)
- J4 pad 6: Net-(J3-Pad6) -> Net-(J3-Pad8)
- J4 pad 8: Net-(J3-Pad8) -> Net-(J3-Pad6)
- J4 pad 9: Net-(J3-Pad9) -> Net-(J3-Pad5)
Routing:
- net Net-(J1-Pad20): track 6.13 -> 5.00 mm
- net Net-(J3-Pad9): track 6.10 -> 5.00 mm
- net Net-(J3-Pad8): track 6.10 -> 5.00 mm
- net Net-(J3-Pad7): track 6.10 -> 5.00 mm
- net Net-(J3-Pad6): track 6.10 -> 5.00 mm
- net Net-(J3-Pad5): track 6.10 -> 5.00 mm
- net Net-(J3-Pad4): track 6.10 -> 5.00 mm
- net Net-(J3-Pad3): track 6.10 -> 5.00 mm
- net Net-(J3-Pad25): track 3.90 -> 5.00 mm
- net Net-(J3-Pad24): track 3.90 -> 5.00 mm
- net Net-(J3-Pad23): track 3.90 -> 5.00 mm
- net Net-(J3-Pad22): track 3.90 -> 5.00 mm
- net Net-(J3-Pad21): track 3.90 -> 5.00 mm
- net Net-(J3-Pad20): track 3.90 -> 5.00 mm
- net Net-(J3-Pad2): track 6.10 -> 5.00 mm
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Other:
- board text added: "Ambient Pressure Side MicroD_Vacuum_Feedthrough_Double_kf40_Reversed Ryan Morgenstern 1/18/23"
- board text added: "Vacuum Side MicroD_Vacuum_Feedthrough_Double_kf40_Reversed Ryan Morgenstern 1/18/23"
- board text removed: "Ambient Pressure Side MicroD_Vacuum_Feedthrough_Double_kf40 Ryan Morgenstern 9/20/22"
- board text removed: "Vacuum Side MicroD_Vacuum_Feedthrough_Double_kf40 Ryan Morgenstern 9/20/22"
