File: KF40-Micro-D_25_Double_Feedthrough/Double_MicroD_25_Gateway - Reversed/Double_MicroD_25_Gateway.kicad_sch (KiCad schematic)
At the start: 4 parts, among them J1 DB25_Female, J2 DB25_Female, J3 DB25_Female, J4 DB25_Female

Commit message: updated kf40- reversed
Connections:
- net at J2.1: now also J1.13; no longer J1.1
- net at J2.10: now also J1.4; no longer J1.10
- net at J2.11: now also J1.3; no longer J1.11
- net at J2.12: now also J1.2; no longer J1.12
- net at J2.13: now also J1.1; no longer J1.13
- net at J2.14 (P14): now also J1.25 (P25); no longer J1.14 (P14)
- net at J2.15 (P15): now also J1.24 (P24); no longer J1.15 (P15)
- net at J2.16 (P16): now also J1.23 (P23); no longer J1.16 (P16)
- net at J2.17 (P17): now also J1.22 (P22); no longer J1.17 (P17)
- net at J2.18 (P18): now also J1.21 (P21); no longer J1.18 (P18)
- net at J2.19 (P19): now also J1.20 (P20); no longer J1.19 (P19)
- net at J2.2: now also J1.12; no longer J1.2
- net at J2.20 (P20): now also J1.19 (P19); no longer J1.20 (P20)
- net at J2.21 (P21): now also J1.18 (P18); no longer J1.21 (P21)
- net at J2.22 (P22): now also J1.17 (P17); no longer J1.22 (P22)
- net at J2.23 (P23): now also J1.16 (P16); no longer J1.23 (P23)
- net at J2.24 (P24): now also J1.15 (P15); no longer J1.24 (P24)
- net at J2.25 (P25): now also J1.14 (P14); no longer J1.25 (P25)
- net at J2.3: now also J1.11; no longer J1.3
- net at J2.4: now also J1.10; no longer J1.4
- net at J2.5: now also J1.9; no longer J1.5
- net at J2.6: now also J1.8; no longer J1.6
- net at J2.8: now also J1.6; no longer J1.8
- net at J2.9: now also J1.5; no longer J1.9
- net at J4.1: now also J3.13; no longer J3.1
- net at J4.10: now also J3.4; no longer J3.10
- net at J4.11: now also J3.3; no longer J3.11
- net at J4.12: now also J3.2; no longer J3.12
- net at J4.13: now also J3.1; no longer J3.13
- net at J4.14 (P14): now also J3.25 (P25); no longer J3.14 (P14)
- net at J4.15 (P15): now also J3.24 (P24); no longer J3.15 (P15)
- net at J4.16 (P16): now also J3.23 (P23); no longer J3.16 (P16)
- net at J4.17 (P17): now also J3.22 (P22); no longer J3.17 (P17)
- net at J4.18 (P18): now also J3.21 (P21); no longer J3.18 (P18)
- net at J4.19 (P19): now also J3.20 (P20); no longer J3.19 (P19)
- net at J4.2: now also J3.12; no longer J3.2
- net at J4.20 (P20): now also J3.19 (P19); no longer J3.20 (P20)
- net at J4.21 (P21): now also J3.18 (P18); no longer J3.21 (P21)
- net at J4.22 (P22): now also J3.17 (P17); no longer J3.22 (P22)
- net at J4.23 (P23): now also J3.16 (P16); no longer J3.23 (P23)
- net at J4.24 (P24): now also J3.15 (P15); no longer J3.24 (P24)
- net at J4.25 (P25): now also J3.14 (P14); no longer J3.25 (P25)
- net at J4.3: now also J3.11; no longer J3.3
- net at J4.4: now also J3.10; no longer J3.4
- net at J4.5: now also J3.9; no longer J3.5
- net at J4.6: now also J3.8; no longer J3.6
- net at J4.8: now also J3.6; no longer J3.8
- net at J4.9: now also J3.5; no longer J3.9
Other:
- moved on the sheet: J2, J4
Changed lines of the file:
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@@
 (kicad_sch (version 20211123) (generator eeschema)
   (paper "A4")
-  (junction (at 153.67 55.88) (diameter 0) (color 0 0 0 0)
-  )
-  (junction (at 193.04 55.88) (diameter 0) (color 0 0 0 0)
-  )
-  (wire (pts (xy 153.67 55.88) (xy 153.67 57.15))
-    (stroke (width 0) (type default) (color 0 0 0 0))
-  )
   (wire (pts (xy 146.05 55.88) (xy 146.05 57.15))
     (stroke (width 0) (type default) (color 0 0 0 0))
   )
-  (wire (pts (xy 193.04 55.88) (xy 153.67 55.88))
-    (stroke (width 0) (type default) (color 0 0 0 0))
-  )
-  (wire (pts (xy 153.67 55.88) (xy 146.05 55.88))
-    (stroke (width 0) (type default) (color 0 0 0 0))
-  )
-  (wire (pts (xy 193.04 55.88) (xy 200.66 55.88))
-    (stroke (width 0) (type default) (color 0 0 0 0))
-  )
-  (symbol (lib_name "DB25_Female_1") (lib_id "Connector:DB25_Female") (at 157.48 95.25 0) (unit 1)
-    (in_bom yes) (on_board yes)
-    (property "Reference" "J2" (id 0) (at 162.052 94.0816 0)
-      (effects (font (size 1.27 1.27)) (justify left))
-    )
-    (property "Value" "DB25_Female" (id 1) (at 162.052 96.393 0)
+  (symbol (lib_name "DB25_Female_1") (lib_id "Connector:DB25_Female") (at 157.48 95.25 0) (mirror x) (unit 1)
+    (in_bom yes) (on_board yes)
+    (property "Reference" "J2" (id 0) (at 162.052 96.4184 0)
+      (effects (font (size 1.27 1.27)) (justify left))
+    )
+    (property "Value" "DB25_Female" (id 1) (at 162.052 94.107 0)
       (effects (font (size 1.27 1.27)) (justify left))
     )
@@
     (pin "GND")
   )
-  (symbol (lib_id "Connector:DB25_Female") (at 204.47 93.98 0) (unit 1)
-    (in_bom yes) (on_board yes)
-    (property "Reference" "J4" (id 0) (at 209.042 92.8116 0)
-      (effects (font (size 1.27 1.27)) (justify left))
-    )
-    (property "Value" "DB25_Female" (id 1) (at 209.042 95.123 0)
+  (symbol (lib_id "Connector:DB25_Female") (at 204.47 93.98 0) (mirror x) (unit 1)
+    (in_bom yes) (on_board yes)
+    (property "Reference" "J4" (id 0) (at 209.042 95.1484 0)
+      (effects (font (size 1.27 1.27)) (justify left))
+    )
+    (property "Value" "DB25_Female" (id 1) (at 209.042 92.837 0)
       (effects (font (size 1.27 1.27)) (justify left))
     )
@@
     (pin "GND")
   )
+  (symbol (lib_id "power:GND") (at 146.05 55.88 180) (unit 1)
+    (in_bom yes) (on_board yes) (fields_autoplaced)
+    (property "Reference" "#PWR?" (id 0) (at 146.05 49.53 0)
+      (effects (font (size 1.27 1.27)) hide)
+    )
+    (property "Value" "GND" (id 1) (at 146.05 52.3042 0))
+    (property "Footprint" "" (id 2) (at 146.05 55.88 0)
+      (effects (font (size 1.27 1.27)) hide)
+    )
+    (property "Datasheet" "" (id 3) (at 146.05 55.88 0)
+      (effects (font (size 1.27 1.27)) hide)
+    )
+    (pin "1")
+  )
   (symbol (lib_id "power:GND") (at 193.04 55.88 180) (unit 1)
     (in_bom yes) (on_board yes) (fields_autoplaced)
@@
     )
     (property "Datasheet" "" (id 3) (at 193.04 55.88 0)
+      (effects (font (size 1.27 1.27)) hide)
+    )
+    (pin "1")
+  )
+  (symbol (lib_id "power:GND") (at 200.66 132.08 0) (unit 1)
+    (in_bom yes) (on_board yes) (fields_autoplaced)
+    (property "Reference" "#PWR?" (id 0) (at 200.66 138.43 0)
+      (effects (font (size 1.27 1.27)) hide)
+    )
+    (property "Value" "GND" (id 1) (at 202.565 133.7838 0)
+      (effects (font (size 1.27 1.27)) (justify left))
+    )
+    (property "Footprint" "" (id 2) (at 200.66 132.08 0)
+      (effects (font (size 1.27 1.27)) hide)
+    )
+    (property "Datasheet" "" (id 3) (at 200.66 132.08 0)
+      (effects (font (size 1.27 1.27)) hide)
+    )
+    (pin "1")
+  )
+  (symbol (lib_id "power:GND") (at 153.67 133.35 0) (unit 1)
+    (in_bom yes) (on_board yes) (fields_autoplaced)
+    (property "Reference" "#PWR?" (id 0) (at 153.67 139.7 0)
+      (effects (font (size 1.27 1.27)) hide)
+    )
+    (property "Value" "GND" (id 1) (at 155.575 135.0538 0)
+      (effects (font (size 1.27 1.27)) (justify left))
+    )
+    (property "Footprint" "" (id 2) (at 153.67 133.35 0)
+      (effects (font (size 1.27 1.27)) hide)
+    )
+    (property "Datasheet" "" (id 3) (at 153.67 133.35 0)
       (effects (font (size 1.27 1.27)) hide)
     )
@@
       (reference "#PWR01") (unit 1) (value "GND") (footprint "")
     )
+    (path "/45ca8cbd-98d6-483f-ab89-fbd2a566d099"
+      (reference "#PWR?") (unit 1) (value "GND") (footprint "")
+    )
+    (path "/6b00c528-113e-49d9-83fe-33b49f38e99a"
+      (reference "#PWR?") (unit 1) (value "GND") (footprint "")
+    )
+    (path "/ff6191a1-3eb9-4b0c-97b1-034f1d6fdcc8"
+      (reference "#PWR?") (unit 1) (value "GND") (footprint "")
+    )
     (path "/00000000-0000-0000-0000-000062d21d3e"
