File: KF40-Micro-D_25_Double_Feedthrough/Double_MicroD_25_Gateway - Reversed/Double_MicroD_25_Gateway.sch (KiCad schematic (older format))
At the start: 4 parts, among them J1 DB25_Female, J2 DB25_Female, J3 DB25_Female, J4 DB25_Female

Commit message: updated kf40- reversed
Connections:
- net at J2.1: now also J1.13; no longer J1.1
- net at J2.10: now also J1.4; no longer J1.10
- net at J2.11: now also J1.3; no longer J1.11
- net at J2.12: now also J1.2; no longer J1.12
- net at J2.13: now also J1.1; no longer J1.13
- net at J2.14 (P14): now also J1.25 (P25); no longer J1.14 (P14)
- net at J2.15 (P15): now also J1.24 (P24); no longer J1.15 (P15)
- net at J2.16 (P16): now also J1.23 (P23); no longer J1.16 (P16)
- net at J2.17 (P17): now also J1.22 (P22); no longer J1.17 (P17)
- net at J2.18 (P18): now also J1.21 (P21); no longer J1.18 (P18)
- net at J2.19 (P19): now also J1.20 (P20); no longer J1.19 (P19)
- net at J2.2: now also J1.12; no longer J1.2
- net at J2.20 (P20): now also J1.19 (P19); no longer J1.20 (P20)
- net at J2.21 (P21): now also J1.18 (P18); no longer J1.21 (P21)
- net at J2.22 (P22): now also J1.17 (P17); no longer J1.22 (P22)
- net at J2.23 (P23): now also J1.16 (P16); no longer J1.23 (P23)
- net at J2.24 (P24): now also J1.15 (P15); no longer J1.24 (P24)
- net at J2.25 (P25): now also J1.14 (P14); no longer J1.25 (P25)
- net at J2.3: now also J1.11; no longer J1.3
- net at J2.4: now also J1.10; no longer J1.4
- net at J2.5: now also J1.9; no longer J1.5
- net at J2.6: now also J1.8; no longer J1.6
- net at J2.8: now also J1.6; no longer J1.8
- net at J2.9: now also J1.5; no longer J1.9
- net at J4.1: now also J3.13; no longer J3.1
- net at J4.10: now also J3.4; no longer J3.10
- net at J4.11: now also J3.3; no longer J3.11
- net at J4.12: now also J3.2; no longer J3.12
- net at J4.13: now also J3.1; no longer J3.13
- net at J4.14 (P14): now also J3.25 (P25); no longer J3.14 (P14)
- net at J4.15 (P15): now also J3.24 (P24); no longer J3.15 (P15)
- net at J4.16 (P16): now also J3.23 (P23); no longer J3.16 (P16)
- net at J4.17 (P17): now also J3.22 (P22); no longer J3.17 (P17)
- net at J4.18 (P18): now also J3.21 (P21); no longer J3.18 (P18)
- net at J4.19 (P19): now also J3.20 (P20); no longer J3.19 (P19)
- net at J4.2: now also J3.12; no longer J3.2
- net at J4.20 (P20): now also J3.19 (P19); no longer J3.20 (P20)
- net at J4.21 (P21): now also J3.18 (P18); no longer J3.21 (P21)
- net at J4.22 (P22): now also J3.17 (P17); no longer J3.22 (P22)
- net at J4.23 (P23): now also J3.16 (P16); no longer J3.23 (P23)
- net at J4.24 (P24): now also J3.15 (P15); no longer J3.24 (P24)
- net at J4.25 (P25): now also J3.14 (P14); no longer J3.25 (P25)
- net at J4.3: now also J3.11; no longer J3.3
- net at J4.4: now also J3.10; no longer J3.4
- net at J4.5: now also J3.9; no longer J3.5
- net at J4.6: now also J3.8; no longer J3.6
- net at J4.8: now also J3.6; no longer J3.8
- net at J4.9: now also J3.5; no longer J3.9
Changed lines of the file:
@@
 F 3 " ~" H 6200 3750 50  0001 C CNN
 	1    6200 3750
-	1    0    0    -1
+	1    0    0    1
 $EndComp
 $Comp
@@
 F 3 " ~" H 8050 3700 50  0001 C CNN
 	1    8050 3700
-	1    0    0    -1
+	1    0    0    1
 $EndComp
 $Comp
